File: Front Plate.kicad_pcb (KiCad board)
At the start: 2 copper layers, 30.2 x 24.9 mm, 4 parts

Commit message: not sure what changes I made
Parts:
- moved   6.14 mm to (143.8, 70.7)
- moved   6.14 mm to (166.2, 70.7)
- moved   6.14 mm to (166.2, 54.3)
- moved   6.14 mm to (143.8, 54.3)
Changed lines of the file:
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@@
   )
   (module MountingHole:MountingHole_3.2mm_M3 (layer F.Cu)
-    (at 160.0277 54.4275)
+    (at 166.16655 54.27)
     (descr "Mounting Hole 3.2mm, no annular, M3")
     (tags "mounting hole 3.2mm no annular m3")
@@
   )
   (module MountingHole:MountingHole_3.2mm_M3 (layer F.Cu)
-    (at 149.9723 54.4275)
+    (at 143.83345 54.27)
     (descr "Mounting Hole 3.2mm, no annular, M3")
     (tags "mounting hole 3.2mm no annular m3")
@@
   )
   (module MountingHole:MountingHole_3.2mm_M3 (layer F.Cu)
-    (at 149.9723 70.57)
+    (at 143.83345 70.73)
     (descr "Mounting Hole 3.2mm, no annular, M3")
     (tags "mounting hole 3.2mm no annular m3")
@@
   )
   (module MountingHole:MountingHole_3.2mm_M3 (layer F.Cu)
-    (at 160.0277 70.57)
+    (at 166.16655 70.73)
     (descr "Mounting Hole 3.2mm, no annular, M3")
     (tags "mounting hole 3.2mm no annular m3")
